File: Hardware/CAD/N32B_v1.2/N32B.kicad_pcb (KiCad board)
At the start: 2 copper layers, 200 x 130 mm, 51 parts, among them IC1 MAX7219CNG, J1 AudioJack4

Commit message: Hardware upgrades
Parts:
- added D1: 1N914, shik:D_DO-35_SOD27_P7.62mm_Horizontal, F.Cu at (198.8, 113.5)
- added G***: LOGO, N32B:n32b-main-board-graphics-v1.2, F.Cu at (128.5, 87.1)
- added J2: AudioJack4, shik:Jack_3.5mm_Horizontal, F.Cu at (221.2, 99.6)
- added R3: 220, Resistors:AXIAL-0.3-KIT, F.Cu at (202.8, 100.7)
- added R4: 4.7k, Resistors:AXIAL-0.3-KIT, F.Cu at (201.1, 137.7)
- added R5: 220, Resistors:AXIAL-0.3-KIT, F.Cu at (199.8, 97.3)
- added RESET1: MOMENTARY-SWITCH-SPST-PTH-6.0MM, Switches:TACTILE_SWITCH_PTH_6.0MM, F.Cu at (200.9, 55.3)
- added U1: 6N138, shik:6n138, F.Cu at (201.2, 123.2)
- B1: footprint shik:SPARKFUN_PRO_MICRO -> shik:ARDUINO_PRO_MICRO
Connections:
- B1 pad 2: Net-(B1-Pad2) -> RX
- B1 pad 22: Net-(B1-Pad22) -> RST
Routing:
- net RX: track 0.00 -> 111.6 mm
- net Net-(D1-Pad2): track 0.00 -> 29.6 mm
- net Net-(D1-Pad1): track 0.00 -> 24.2 mm
- net RST: track 0.00 -> 17.1 mm
- net Net-(J2-PadR1): track 0.00 -> 16.2 mm
- net Net-(R4-PadP$1): track 0.00 -> 13.2 mm
- net R16: track 43.6 -> 47.1 mm
- net R32: track 95.9 -> 99.0 mm
- net R28: track 91.8 -> 93.0 mm
- net R20: track 65.7 -> 66.8 mm
- net R24: track 69.8 -> 70.8 mm
- net R14: track 34.6 -> 35.5 mm
- net SEGF: track 38.9 -> 39.5 mm
- net SEGG: track 49.7 -> 50.2 mm
- net SEGA: track 36.6 -> 37.1 mm
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Other:
- outline, holes or cut-outs redrawn
