File: Hardware/CAD/N32B_v1.2/N32B.sch (KiCad schematic (older format))
At the start: 51 parts, among them IC1 MAX7219CNG, J1 AudioJack4

Commit message: Hardware upgrades
Parts:
- added D1: 1N914, shik:D_DO-35_SOD27_P7.62mm_Horizontal, symbol Diode:1N914
- added J2: AudioJack4, shik:Jack_3.5mm_Horizontal, symbol Connector:AudioJack4
- added R3, R5: 220, Resistors:AXIAL-0.3-KIT, symbol SparkFun-Resistors:10KOHM-HORIZ_KIT-1_4W-5%
- added R4: 4.7k, Resistors:AXIAL-0.3-KIT, symbol SparkFun-Resistors:10KOHM-HORIZ_KIT-1_4W-5%
- added RESET1: MOMENTARY-SWITCH-SPST-PTH-6.0MM, Switches:TACTILE_SWITCH_PTH_6.0MM, symbol SparkFun-Switches:MOMENTARY-SWITCH-SPST-PTH-6.0MM
- added U1: 6N138, shik:6n138, symbol Isolator:6N138
- B1: footprint shik:SPARKFUN_PRO_MICRO -> shik:ARDUINO_PRO_MICRO; symbol SparkFun-Boards:SPARKFUN_PRO_MICRO -> Shik-Tech:ARDUINO_PRO_MICRO
Connections:
- net GND: now also R4.P$2 (2), RESET1.3 (2), U1.5 (GND)
- net VCC: now also R5.P$1 (1), U1.8 (VCC)
- net RX: now reaches B1.2 (RXI)
- net RX: now also R5.P$2 (2), U1.6 (VO2)
- net RST: now reaches B1.22 (RST)
- net RST: now also RESET1.1
- new net: J2.R1, R3.P$1 (1)
- new net: D1.2 (A), J2.T, U1.3 (C2)
- new net: D1.1 (K), R3.P$2 (2), U1.2 (C1)
- new net: R4.P$1 (1), U1.7 (VO1)
Other:
- moved on the sheet: B1, C1, C2, Display1, H1, H2, H3, H4, H5, H6, IC1, J1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
